File: kicad/vscp-din-m1-wireless-p1/vanilla-vscp-din-m1.kicad_pcb (KiCad board)
At the start: 2 copper layers, 64.8 x 51 mm, 3 parts, among them J1 Conn_01x04_Left, J2 Conn_01x04_Right, J3 Conn_01x06

Commit message: Updated design files
Other:
- net class Default removed
