File: kicad/vscp-din-m1-wireless-p1/vscp-din-wireless-esp32.kicad_pcb (KiCad board)
At the start: 2 copper layers, 64.8 x 51 mm, 3 parts, among them J1 Conn_01x04_Left, J2 Conn_01x04_Right, J3 Conn_01x06

Commit message: Fixed power
Parts:
- added REF**: PhoenixContact_MCV_1,5_12-GF-3.81_1x12_P3.81mm_Vertical_Thr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, Connector_Phoenix_MC:PhoenixContact_MCV_1,5_12-GF-3.81_1x12_P3.81mm_Vertical_ThreadedFlange, F.Cu at (128.3, 85.3)
- added REF**: TerminalBlock_4Ucon_1x12_P3.50mm_Vertical, TerminalBlock_4Ucon:TerminalBlock_4Ucon_1x12_P3.50mm_Vertical, F.Cu at (133.6, 70.9)

Commit message: Updated design files
Other:
- net class Default removed
